File: Circuit/AllInOneModule/AllInOneModule.kicad_pcb (KiCad board)
At the start: 2 copper layers, 40 parts, among them J101 Servo, J102 KeyPad, Q3 DMG3415U, SW1 KMR2, SW2 KMR2, U1 ESP32-S3-MINI-1, U101 HT16K33, U2 AP2112/RT9080-3.3, U3 MCP73831T-2ACI/OT, X1 JSTPH, X3 USB C

Commit message: Snapshot commit.
Parts:
- C8: value C -> 10µF
- J101: footprint Connector_PinHeader_2.54mm:PinHeader_1x03_P2.54mm_Vertical -> Connector_PinHeader_2.54mm:PinHeader_1x03_P2.54mm_Horizontal
- J102: footprint Connector_PinHeader_2.54mm:PinHeader_1x07_P2.54mm_Vertical -> Connector_PinHeader_2.54mm:PinHeader_1x07_P2.54mm_Horizontal
- SW1: value KMR2 -> BOOT0
- SW2: value KMR2 -> RESET
- moved H102 152.2 mm to (266.7, 72.4)
- moved DI104 149.8 mm to (247.7, 53.3)
- moved H101 130.4 mm to (266.7, 35.6)
- moved DI102 125.3 mm to (196.8, 53.3)
- moved DI103 124.4 mm to (222.2, 53.3)
- moved X1 105.4 mm to (161.3, 36.8), turned to 180 degrees
- moved C101 100.0 mm to (158.0, 53.3), turned to -90 degrees
- moved DI101 99.9 mm to (171.4, 53.3)
- moved Q3 87.9 mm to (133.9, 47.0)
- moved U3 83.4 mm to (152.4, 38.7), turned to 180 degrees
- moved R4 83.1 mm to (148.6, 39.9)
- moved CHG0 80.2 mm to (158.8, 41.2)
- moved R5 79.7 mm to (138.4, 43.2), turned to 90 degrees
- moved C3 79.6 mm to (157.5, 37.7), turned to -90 degrees
- moved SW1 77.6 mm to (118.6, 52.5)
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Connections:
- net /D11 renamed /C3
- net /D5 renamed /C1
- net /D9 renamed /C2
- net /MOSI renamed /LockServo
- net 3.3V renamed +3V3
Routing:
- net /Display Module/B: track 0.00 -> 205.1 mm, vias 0 -> 5
- net /Display Module/A: track 0.00 -> 193.4 mm, vias 0 -> 5
- net /Display Module/DP: track 0.00 -> 190.1 mm, vias 0 -> 5
- net /Display Module/N: track 0.00 -> 180.1 mm, vias 0 -> 5
- net /Display Module/M: track 0.00 -> 166.1 mm, vias 0 -> 5
- net /Display Module/K: track 0.00 -> 165.1 mm, vias 0 -> 5
- net /Display Module/J: track 0.00 -> 158.8 mm, vias 0 -> 5
- net /Display Module/L: track 0.00 -> 158.4 mm, vias 0 -> 5
- net /Display Module/H: track 0.00 -> 148.6 mm, vias 0 -> 5
- net /Display Module/F: track 0.00 -> 137.4 mm, vias 0 -> 5
- net /Display Module/G2: track 0.00 -> 131.5 mm, vias 0 -> 5
- net /Display Module/G1: track 0.00 -> 128.3 mm, vias 0 -> 5
- net /Display Module/COM7: track 0.00 -> 127.4 mm, vias 0 -> 2
- net /Display Module/E: track 0.00 -> 125.4 mm, vias 0 -> 5
- net /Display Module/D: track 0.00 -> 120.9 mm, vias 0 -> 5
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Other:
- board outline added: 176.5 x 44.5 mm

Commit message: Snapshot commit.
Parts:
- moved C1 30.6 mm to (125.9, 48.3)
- moved SW1 14.6 mm to (109.3, 41.2)
- moved R101 7.49 mm to (126.1, 72.2), turned to 90 degrees
- moved C3 6.27 mm to (153.2, 42.3)
- moved R102 5.82 mm to (126.1, 67.5), turned to 90 degrees
- moved R1 5.37 mm to (112.1, 66.6)
- moved C4 3.77 mm to (109.6, 67.5), turned to -90 degrees
- moved CHG0 3.43 mm to (156.3, 43.6)
- moved R4 3.32 mm to (151.2, 42.0), turned to 90 degrees
- moved SW2 2.95 mm to (105.8, 67.5)
- moved R12 2.55 mm to (130.6, 43.1)
- moved C2 2.17 mm to (121.6, 45.4)
- moved C8 1.91 mm to (123.6, 45.4)
- moved C10 1.58 mm to (98.8, 67.1)
- moved C7 1.25 mm to (96.4, 67.0)
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Routing:
- net GND: track 6.74 -> 112.1 mm, vias 1 -> 14
- net VBUS: track 0.00 -> 93.3 mm, vias 0 -> 7
- net /SCL: track 0.00 -> 72.0 mm, vias 0 -> 3
- net /D-: track 0.00 -> 71.3 mm, vias 0 -> 4
- net /SDA: track 0.00 -> 62.9 mm, vias 0 -> 3
- net /D+: track 0.00 -> 62.1 mm, vias 0 -> 4
- net VBAT: track 0.00 -> 55.1 mm, vias 0 -> 4
- net /C1: track 0.00 -> 47.2 mm, vias 0 -> 3
- net /D6: track 0.00 -> 46.3 mm, vias 0 -> 4
- net /C2: track 0.00 -> 33.5 mm, vias 0 -> 4
- net /D10: track 0.00 -> 29.0 mm, vias 0 -> 2
- net /C3: track 0.00 -> 27.8 mm, vias 0 -> 2
- net /D13: track 0.00 -> 26.0 mm, vias 0 -> 2
- net /D12: track 0.00 -> 25.9 mm, vias 0 -> 2
- net /LockServo: track 0.00 -> 25.5 mm, vias 0 -> 1
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- added copper zone on F.Cu, net +3V3
- added copper zone on B.Cu, net GND

Commit message: Snapshot commit.
Parts:
- moved X3 0.98 mm to (139.8, 35.8)
Routing:
- net VBUS: track 93.3 -> 104.7 mm
- net GND: track 112.1 -> 122.7 mm
- net /BOOT0: track 10.9 -> 8.55 mm
- net /D+: track 62.1 -> 64.2 mm
- net Net-(R8-Pad2): track 1.93 -> 2.92 mm
- net Net-(R5-Pad2): track 2.12 -> 3.08 mm
- net VBAT: track 55.1 -> 56.0 mm

Commit message: Snapshot commit.
Parts:
- moved X3 1.02 mm to (140.8, 35.7)
- moved R5 1.02 mm to (139.4, 43.1)
- moved R8 1.02 mm to (142.0, 43.1)
Routing:
- net GND: track 122.7 -> 123.4 mm

Commit message: Snapshot commit.
Routing:
- net /Display Module/L: track 158.4 -> 157.4 mm
- net /Display Module/M: track 166.1 -> 165.1 mm
- net /Display Module/DP: track 187.6 -> 188.3 mm
