File: Circuit/AllInOneModule/AllInOneModule.kicad_pcb (KiCad board)
At the start: 2 copper layers, 176.5 x 44.5 mm, 40 parts, among them J101 Servo, J102 KeyPad, Q3 DMG3415U, SW1 BOOT0, SW2 RESET, U1 ESP32-S3-MINI-1, U101 HT16K33, U2 AP2112/RT9080-3.3, U3 MCP73831T-2ACI/OT, X1 JSTPH, X3 USB C

Commit message: Snapshot commit.
Routing:
- net GND: track 123.8 -> 121.9 mm

Commit message: Snapshot commit.
Parts:
- CHG0: value ORANGE -> Charge
- X1: value JSTPH -> Battery
Changed lines of the file:
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@@
     (property "Sheetname" "")
     (attr smd)
-    (fp_text reference "R4" (at 0 -1.43 90) (layer "F.SilkS")
-      (effects (font (size 1 1) (thickness 0.15)))
-    )
-    (fp_text value "5.1K" (at 0 1.43 90) (layer "F.Fab")
-      (effects (font (size 1 1) (thickness 0.15)))
+    (fp_text reference "R4" (at -0.063 0.0508 90) (layer "F.SilkS")
+      (effects (font (size 0.5 0.5) (thickness 0.075)))
+    )
+    (fp_text value "5.1K" (at -0.0122 -1.0668 90) (layer "F.Fab")
+      (effects (font (size 0.5 0.5) (thickness 0.075)))
     )
     (fp_text user "${REFERENCE}" (at 0 0 90) (layer "F.Fab")
@@
     (property "Sheetname" "")
     (attr through_hole)
-    (fp_text reference "J102" (at -4.2598 -0.5726 90) (layer "F.SilkS")
-      (effects (font (size 1 1) (thickness 0.15)))
-    )
-    (fp_text value "KeyPad" (at 4.385 17.51 90) (layer "F.Fab")
+    (fp_text reference "J102" (at -4.2598 -0.5726 90) (layer "F.Fab")
+      (effects (font (size 1 1) (thickness 0.15)))
+    )
+    (fp_text value "KeyPad" (at -2.2278 13.4482 180) (layer "F.SilkS")
       (effects (font (size 1 1) (thickness 0.15)))
     )
@@
     (property "Sheetname" "")
     (attr smd)
-    (fp_text reference "U3" (at 0 -2.4) (layer "F.SilkS")
-      (effects (font (size 1 1) (thickness 0.15)))
-    )
-    (fp_text value "MCP73831T-2ACI/OT" (at 0 2.4) (layer "F.Fab")
+    (fp_text reference "U3" (at 0 0) (layer "F.SilkS")
+      (effects (font (size 0.5 0.5) (thickness 0.075)))
+    )
+    (fp_text value "MCP73831T-2ACI/OT" (at 3.6068 -0.6592 90) (layer "F.Fab")
       (effects (font (size 1 1) (thickness 0.15)))
     )
@@
     (property "Sheetname" "")
     (attr smd)
-    (fp_text reference "X1" (at 0 -5.8) (layer "F.SilkS")
-      (effects (font (size 1 1) (thickness 0.15)))
-    )
-    (fp_text value "JSTPH" (at -5.08 5.24) (layer "F.Fab")
+    (fp_text reference "X1" (at 0 -5.8) (layer "F.Fab")
+      (effects (font (size 1 1) (thickness 0.15)))
+    )
+    (fp_text value "Battery" (at -5.842 0.9144 90) (layer "F.SilkS")
       (effects (font (size 1 1) (thickness 0.15)))
     )
@@
     (property "Sheetname" "")
     (attr smd)
-    (fp_text reference "CHG0" (at 0 -1.43) (layer "F.SilkS")
-      (effects (font (size 1 1) (thickness 0.15)))
-    )
-    (fp_text value "ORANGE" (at 0 1.43) (layer "F.Fab")
+    (fp_text reference "CHG0" (at 0.0763 0 90) (layer "F.Fab")
+      (effects (font (size 0.5 0.5) (thickness 0.075)))
+    )
+    (fp_text value "Charge" (at 0.4319 1.6256 180) (layer "F.SilkS")
       (effects (font (size 1 1) (thickness 0.15)))
     )
@@
     (property "Sheetname" "")
     (attr smd)
-    (fp_text reference "R2" (at 0 -1.43 90) (layer "F.SilkS")
-      (effects (font (size 1 1) (thickness 0.15)))
-    )
-    (fp_text value "5.1K" (at 0 1.43 90) (layer "F.Fab")
-      (effects (font (size 1 1) (thickness 0.15)))
+    (fp_text reference "R2" (at 0 0 90) (layer "F.SilkS")
+      (effects (font (size 0.5 0.5) (thickness 0.075)))
+    )
+    (fp_text value "5.1K" (at -0.0508 1.2192 90) (layer "F.Fab")
+      (effects (font (size 0.5 0.5) (thickness 0.075)))
     )
     (fp_text user "${REFERENCE}" (at 0 0 90) (layer "F.Fab")
@@
       (effects (font (size 1 1) (thickness 0.15)))
     )
-    (fp_text value "MountingHole" (at 0 4.2) (layer "F.Fab")
+    (fp_text value "MountingHole" (at 0 4.2) (layer "F.Fab") hide
       (effects (font (size 1 1) (thickness 0.15)))
     )
@@
     (property "Sheetname" "")
     (attr through_hole)
-    (fp_text reference "J101" (at 4.385 -2.27 90) (layer "F.SilkS")
-      (effects (font (size 1 1) (thickness 0.15)))
-    )
-    (fp_text value "Servo" (at 4.385 7.35 90) (layer "F.Fab")
+    (fp_text reference "J101" (at 4.385 -2.27 90) (layer "F.Fab")
+      (effects (font (size 1 1) (thickness 0.15)))
+    )
+    (fp_text value "Servo" (at -2.5326 -0.2894 180) (layer "F.SilkS")
       (effects (font (size 1 1) (thickness 0.15)))
     )
@@
     (property "Sheetname" "")
     (attr smd)
-    (fp_text reference "C3" (at 0 -1.68 90) (layer "F.SilkS")
-      (effects (font (size 1 1) (thickness 0.15)))
-    )
-    (fp_text value "10µF" (at 0 1.68 90) (layer "F.Fab")
-      (effects (font (size 1 1) (thickness 0.15)))
+    (fp_text reference "C3" (at 0 0 90) (layer "F.SilkS")
+      (effects (font (size 0.5 0.5) (thickness 0.075)))
+    )
+    (fp_text value "10µF" (at 0.066 -1.2192 90) (layer "F.Fab")
+      (effects (font (size 0.5 0.5) (thickness 0.075)))
     )
     (fp_text user "${REFERENCE}" (at 0 0 90) (layer "F.Fab")
