File: Circuit/AllInOneModule/AllInOneModule.kicad_pcb (KiCad board)
At the start: 2 copper layers, 176.5 x 44.5 mm, 40 parts, among them J101 Servo, J102 KeyPad, Q3 DMG3415U, SW1 BOOT0, SW2 RESET, U1 ESP32-S3-MINI-1, U101 HT16K33, U2 AP2112/RT9080-3.3, U3 MCP73831T-2ACI/OT, X1 Battery, X3 USB C

Commit message: Nearly Complete Circuit Boards.
Changed lines of the file:
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@@
     (pad "2" smd roundrect (at 1 -2.85 180) (size 1 3.5) (layers "F.Cu" "F.Paste" "F.Mask") (roundrect_rratio 0.25)
       (net 3 "VBAT") (pinfunction "2") (pintype "passive"))
-    (pad "MP" smd roundrect (at -3.35 2.9 180) (size 1.5 3.4) (layers "F.Cu" "F.Paste" "F.Mask") (roundrect_rratio 0.166667))
-    (pad "MP" smd roundrect (at 3.35 2.9 180) (size 1.5 3.4) (layers "F.Cu" "F.Paste" "F.Mask") (roundrect_rratio 0.166667))
+    (pad "MP" smd roundrect (at -3.35 2.9 180) (size 1.5 3.4) (layers "F.Cu" "F.Paste" "F.Mask") (roundrect_rratio 0.1666673333))
+    (pad "MP" smd roundrect (at 3.35 2.9 180) (size 1.5 3.4) (layers "F.Cu" "F.Paste" "F.Mask") (roundrect_rratio 0.1666673333))
     (model "${KICAD6_3DMODEL_DIR}/Connector_JST.3dshapes/JST_PH_S2B-PH-K_1x02_P2.00mm_Horizontal.step"
       (offset (xyz -1 1.5 0))
@@
     (pad "3" smd roundrect locked (at 1.1375 0) (size 1.325 0.6) (layers "F.Cu" "F.Paste" "F.Mask") (roundrect_rratio 0.25)
       (net 3 "VBAT") (pinfunction "D") (pintype "passive"))
-    (model "${KICAD6_3DMODEL_DIR}/Package_TO_SOT_SMD.3dshapes/SOT-23-3.wrl"
+    (model "${KICAD6_3DMODEL_DIR}/Package_TO_SOT_SMD.3dshapes/SOT-23.wrl"
       (offset (xyz 0 0 0))
       (scale (xyz 1 1 1))

Commit message: Nearly Complete Circuit Boards.
Routing:
- net /D+: track 64.2 -> 65.2 mm
- net /D-: track 71.1 -> 72.1 mm
Changed lines of the file:
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@@
   (via (at 110.1344 63.9572) (size 0.8) (drill 0.4) (layers "F.Cu" "B.Cu") (net 53))
   (segment (start 119.9388 63.9572) (end 119.9388 63.7463) (width 0.2) (layer "B.Cu") (net 53))
+  (segment (start 139.76515 32.6136) (end 139.81595 32.5628) (width 0.2) (layer "B.Cu") (net 53))
   (segment (start 119.9388 63.7463) (end 119.9896 63.6955) (width 0.2) (layer "B.Cu") (net 53))
   (segment (start 110.1344 63.9572) (end 119.9388 63.9572) (width 0.2) (layer "B.Cu") (net 53))
-  (segment (start 123.698 32.6136) (end 140.4112 32.6136) (width 0.2) (layer "B.Cu") (net 53))
+  (segment (start 123.698 32.6136) (end 139.76515 32.6136) (width 0.2) (layer "B.Cu") (net 53))
+  (segment (start 139.81595 32.5628) (end 141.4272 32.5628) (width 0.2) (layer "B.Cu") (net 53))
   (segment (start 111.2175 60.7223) (end 111.2175 60.703902) (width 0.2) (layer "F.Cu") (net 54))
   (segment (start 139.989266 39.151266) (end 140.0556 39.2176) (width 0.2) (layer "F.Cu") (net 54))
@@
   (via (at 118.9228 61.0108) (size 0.8) (drill 0.4) (layers "F.Cu" "B.Cu") (net 54))
   (segment (start 114.808 61.0108) (end 114.4016 60.6044) (width 0.2) (layer "B.Cu") (net 54))
+  (segment (start 122.7216 33.3136) (end 140.0551 33.3136) (width 0.2) (layer "B.Cu") (net 54))
   (segment (start 122.6312 33.2232) (end 122.7216 33.3136) (width 0.2) (layer "B.Cu") (net 54))
+  (segment (start 140.0551 33.3136) (end 140.1064 33.2623) (width 0.2) (layer "B.Cu") (net 54))
   (segment (start 114.4016 60.6044) (end 111.117998 60.6044) (width 0.2) (layer "B.Cu") (net 54))
   (segment (start 140.1059 33.2628) (end 140.1064 33.2623) (width 0.2) (layer "B.Cu") (net 54))
   (segment (start 118.9228 61.0108) (end 114.808 61.0108) (width 0.2) (layer "B.Cu") (net 54))
-  (segment (start 122.7216 33.3136) (end 139.0899 33.3136) (width 0.2) (layer "B.Cu") (net 54))
   (segment (start 155.4988 42.0238) (end 155.4988 43.5862) (width 0.25) (layer "F.Cu") (net 77))
   (segment (start 155.4988 43.5862) (end 155.4986 43.5864) (width 0.25) (layer "F.Cu") (net 77))

Commit message: Nearly Complete Circuit Boards.
Parts:
- added D101: POWER, LED_SMD:LED_0603_1608Metric, F.Cu at (125.2, 62.6)
- added R103: 30, Resistor_SMD:R_0603_1608Metric, F.Cu at (129.2, 62.6)
Routing:
- net VBUS: track 105.1 -> 101.5 mm
- net Net-(D101-Pad2): track 0.00 -> 2.41 mm
- net GND: track 121.9 -> 120.5 mm
- net VBAT: track 56.0 -> 57.4 mm, vias 4 -> 3
