File: Circuit/AllInOneModule/AllInOneModule.kicad_sch (KiCad schematic)
At the start: 28 parts, among them J101 Servo, J102 KeyPad

Commit message: Snapshot commit.
Parts:
- removed unit 3 of X1
- removed unit 2 of X1
- C1, C2, C7, C9: value (none) -> 10uF; footprint (none) -> Capacitor_SMD:C_0805_2012Metric; MPN (none) -> Samsung Electro-Mechanics CL21A106KQFNFNE; Mouser Part Number (none) -> 187-CL21A106KQFNFNE
- C10, C4: value (none) -> 1uF; footprint (none) -> Capacitor_SMD:C_0603_1608Metric; MPN (none) -> KEMET C0603C105K9PAC7411; Mouser Part Number (none) -> 80-C0603C105K9PLR
- C3, C6, C8: value (none) -> 10µF; footprint (none) -> Capacitor_SMD:C_0805_2012Metric; MPN (none) -> Samsung Electro-Mechanics CL21A106KQFNFNE; Mouser Part Number (none) -> 187-CL21A106KQFNFNE
- CHG0: value (none) -> ORANGE; footprint (none) -> LED_SMD:LED_0603_1608Metric; MPN (none) -> LITEON LTST-C190KFKT; Mouser Part Number (none) -> 859-LTST-C190KFKT
- D4: value (none) -> S5A; footprint (none) -> Extra:S5AE357T; MPN (none) -> Diotec Semiconductor S5A; Mouser Part Number (none) -> 637-S5A
- Q3: value (none) -> DMG3415U; footprint (none) -> Package_TO_SOT_SMD:SOT-23-3; MPN (none) -> Diodes Incorporated DMG3415U-7; Mouser Part Number (none) -> 621-DMG3415U-7
- R1, R2, R4, R5, R8: value (none) -> 5.1K; footprint (none) -> Resistor_SMD:R_0603_1608Metric; MPN (none) -> YAGEO RC0603JR-075K1P; Mouser Part Number (none) -> 603-RC0603JR-075K1P
- R12, R7: value (none) -> 100K; footprint (none) -> Resistor_SMD:R_0603_1608Metric; MPN (none) -> YAGEO RT0603DRD07100KL; Mouser Part Number (none) -> 603-RT0603DRD07100KL
- SW1, SW2: value (none) -> KMR2; footprint (none) -> Button_Switch_SMD:SW_Push_1P1T_NO_CK_KMR2; MPN (none) -> C&K KMR211NG LFS; Mouser Part Number (none) -> 611-KMR211NGLFS
- U1: value (none) -> ESP32-S3-MINI-1; footprint (none) -> ESP32-WROOM:ESP32_S3_WROOM-1; MPN (none) -> Espressif Systems ESP32-S3-MINI-1-N8; Mouser Part Number (none) -> 356-ESP32-S3-MINI1N8
- U2: value (none) -> AP2112/RT9080-3.3; footprint (none) -> Package_TO_SOT_SMD:SOT-23-5; MPN (none) -> Diodes Incorporated AP2112K-3.3TRG1; Mouser Part Number (none) -> 621-AP2112K-3.3TRG1
- U3: value (none) -> MCP73831T-2ACI/OT; footprint (none) -> Package_TO_SOT_SMD:SOT-23-5; MPN (none) -> Microchip Technology MCP73831T-2ACI/OT; Mouser Part Number (none) -> 579-MCP73831T-2ACIOT
- X1: value (none) -> JSTPH; footprint (none) -> Connector_JST:JST_PH_S2B-PH-SM4-TB_1x02-1MP_P2.00mm_Horizontal; MPN (none) -> JST Commercial S2B-PH-SM4-TB(LF)(SN); Mouser Part Number (none) -> 306-S2BPHSM4TBLFSN
- X3: value (none) -> USB C; footprint (none) -> Extra:CONN_USB4930-00-A_GCT; MPN (none) -> GCT USB4930-00-A; Mouser Part Number (none) -> 640-USB4930-00-A
Connections:
- net +3V3: now also U1.2 (3V3); no longer U1.3 (3V3)
- net BOOT0: now also SW1.2 (S1), U1.27 (IO0_BOOT0); no longer SW1.B (S), SW1.B' (S1), U1.4 (IO0_BOOT0)
- net C1: now also U1.5 (IO5); no longer U1.9 (IO5)
- net C2: now also U1.17 (IO9); no longer U1.13 (IO9)
- net C3: now also U1.19 (IO11); no longer U1.15 (IO11)
- net D+: now also U1.14 (IO20/D+); no longer U1.24 (IO20/D+)
- net D-: now also U1.13 (IO19/D-); no longer U1.23 (IO19/D-)
- net D10: now also U1.18 (IO10); no longer U1.14 (IO10)
- net D12: now also U1.20 (IO12); no longer U1.16 (IO12)
- net D13: now also U1.21 (IO13); no longer U1.17 (IO13)
- net D6: now also U1.6 (IO6); no longer U1.10 (IO6)
- net GND: now also SW1.1 (P1), SW2.1 (P1), U1.25 (IO48), U1.40 (GND), U1.EPad (EXP), X3.A1 (GND), X3.A12 (GND), X3.B1 (GND), X3.B12 (GND); no longer SW1.A (P), SW1.A' (P1), SW2.A (P), SW2.A' (P1), U1.2 (GND), U1.30 (IO48), U1.42 (GND), U1.43 (GND), U1.46 (GND), U1.47 (GND), U1.48 (GND), U1.49 (GND), U1.50 (GND), U1.51 (GND), U1.52 (GND), U1.53 (GND), U1.54 (GND), U1.55 (GND), U1.56 (GND), U1.57 (GND), U1.58 (GND), U1.59 (GND), U1.60 (GND), U1.61 (EXP), U1.62 (GND), U1.63 (GND), U1.64 (GND), U1.65 (GND), U1.66 (EXP), U1.67 (EXP), U1.68 (EXP), U1.69 (EXP), U1.70 (EXP), U1.71 (EXP), U1.72 (EXP), U1.73 (EXP), X3.A1B12 (GND), X3.B1A12 (GND)
- net LockServo: now also U1.28 (IO35); no longer U1.31 (IO35)
- net RESET: now also SW2.2 (S1), U1.3 (EN); no longer SW2.B (S), SW2.B' (S1), U1.45 (EN)
- net SCL: now also U1.4 (IO4); no longer U1.8 (IO4)
- net SDA: now also U1.15 (IO3); no longer U1.7 (IO3)
- net VBUS: now also CHG0.2 (A), D4.1 (A), X3.A4 (VBUS), X3.A9 (VBUS), X3.B4 (VBUS), X3.B9 (VBUS); no longer CHG0.A, D4.A, X3.A4B9 (VBUS), X3.B4A9 (VBUS)
- net VHI: now also D4.2 (C); no longer D4.C
- net at R2.1: now also CHG0.1 (C); no longer CHG0.C

Commit message: Snapshot commit.
Parts:
- J101: footprint Connector_PinHeader_2.54mm:PinHeader_1x03_P2.54mm_Vertical -> Connector_PinHeader_2.54mm:PinHeader_1x03_P2.54mm_Horizontal
- J102: footprint Connector_PinHeader_2.54mm:PinHeader_1x07_P2.54mm_Vertical -> Connector_PinHeader_2.54mm:PinHeader_1x07_P2.54mm_Horizontal
- SW1: value KMR2 -> BOOT0
- SW2: value KMR2 -> RESET

Commit message: Snapshot commit.
Parts:
- CHG0: value ORANGE -> Charge
- X1: value JSTPH -> Battery
Changed lines of the file:
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@@
     (in_bom yes) (on_board yes)
     (property "Reference" "CHG0" (id 0) (at 52.07 168.275 0))
-    (property "Value" "ORANGE" (id 1) (at 52.07 175.514 0))
+    (property "Value" "Charge" (id 1) (at 52.07 175.514 0))
     (property "Footprint" "LED_SMD:LED_0603_1608Metric" (id 2) (at 53.34 172.72 0)
       (effects (font (size 1.27 1.27)) hide)
@@
       (effects (font (size 1.27 1.0795)) (justify left bottom))
     )
-    (property "Value" "JSTPH" (id 1) (at 123.19 43.18 90)
+    (property "Value" "Battery" (id 1) (at 123.19 43.18 90)
       (effects (font (size 1.27 1.0795)) (justify left bottom))
     )
@@
     )
     (path "/08d80019-55a3-4b43-ae6e-d4c068102a1f"
-      (reference "CHG0") (unit 1) (value "ORANGE") (footprint "LED_SMD:LED_0603_1608Metric")
+      (reference "CHG0") (unit 1) (value "Charge") (footprint "LED_SMD:LED_0603_1608Metric")
     )
     (path "/b366251b-8404-4292-b10a-09cfc7c147b0"
@@
     )
     (path "/416d7f87-5680-4e19-b7ca-f06b5514af89"
-      (reference "X1") (unit 1) (value "JSTPH") (footprint "Connector_JST:JST_PH_S2B-PH-SM4-TB_1x02-1MP_P2.00mm_Horizontal")
+      (reference "X1") (unit 1) (value "Battery") (footprint "Connector_JST:JST_PH_S2B-PH-SM4-TB_1x02-1MP_P2.00mm_Horizontal")
     )
     (path "/9c7675e4-432d-4544-9546-0b16942bf93d"

Commit message: Nearly Complete Circuit Boards.
Parts:
- J101, J102: now left out of the parts list
Changed lines of the file:
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@@
   )
   (symbol (lib_id "Connector:Conn_01x03_Male") (at 151.765 95.885 180) (unit 1)
-    (in_bom yes) (on_board yes) (fields_autoplaced)
+    (in_bom no) (on_board yes) (fields_autoplaced)
     (property "Reference" "J101" (id 0) (at 153.67 94.6149 0)
       (effects (font (size 1.27 1.27)) (justify right))
@@
   )
   (symbol (lib_id "Connector:Conn_01x07_Male") (at 152.4 111.76 180) (unit 1)
-    (in_bom yes) (on_board yes) (fields_autoplaced)
+    (in_bom no) (on_board yes) (fields_autoplaced)
     (property "Reference" "J102" (id 0) (at 153.67 110.4899 0)
       (effects (font (size 1.27 1.27)) (justify right))

Commit message: Nearly Complete Circuit Boards.
Parts:
- added D101: POWER, LED_SMD:LED_0603_1608Metric, symbol Device:LED
- added R103: 30, Resistor_SMD:R_0603_1608Metric, symbol Device:R
Connections:
- net +3V3: now also R103.1
- net GND: now also D101.1 (K)
- new net: D101.2 (A), R103.2
Changed lines of the file:
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@@
+    (stroke (width 0) (type default) (color 0 0 0 0))
+  )
+  (wire (pts (xy 140.97 32.385) (xy 140.97 34.925))
     (stroke (width 0) (type default) (color 0 0 0 0))
   )
@@
   (label "C1" (at 45.72 109.22 180)
     (effects (font (size 1.27 1.27)) (justify right bottom))
+  )
+  (symbol (lib_id "Device:R") (at 140.97 28.575 0) (unit 1)
+    (in_bom yes) (on_board yes) (fields_autoplaced)
+    (property "Reference" "R103" (id 0) (at 143.51 27.3049 0)
+      (effects (font (size 1.27 1.27)) (justify left))
+    )
+    (property "Value" "30" (id 1) (at 143.51 29.8449 0)
+      (effects (font (size 1.27 1.27)) (justify left))
+    )
+    (property "Footprint" "Resistor_SMD:R_0603_1608Metric" (id 2) (at 139.192 28.575 90)
+      (effects (font (size 1.27 1.27)) hide)
+    )
+    (property "Datasheet" "~" (id 3) (at 140.97 28.575 0)
+      (effects (font (size 1.27 1.27)) hide)
+    )
+    (property "Mouser Part Number" "603-AC0603JR-0730RL " (id 4) (at 140.97 28.575 0)
+      (effects (font (size 1.27 1.27)) hide)
+    )
+    (property "MPN" "YAGEO AC0603JR-0730RL " (id 5) (at 140.97 28.575 0)
+      (effects (font (size 1.27 1.27)) hide)
+    )
+    (pin "1")
+    (pin "2")
   )
   (symbol (lib_id "AllInOneModule-eagle-import:LED0603_NOOUTLINE") (at 53.34 172.72 0) (unit 1)
@@
     (pin "EPad")
   )
+  (symbol (lib_id "Device:LED") (at 140.97 38.735 90) (unit 1)
+    (in_bom yes) (on_board yes) (fields_autoplaced)
+    (property "Reference" "D101" (id 0) (at 144.78 39.0524 90)
+      (effects (font (size 1.27 1.27)) (justify right))
+    )
+    (property "Value" "POWER" (id 1) (at 144.78 41.5924 90)
+      (effects (font (size 1.27 1.27)) (justify right))
+    )
+    (property "Footprint" "LED_SMD:LED_0603_1608Metric" (id 2) (at 140.97 38.735 0)
+      (effects (font (size 1.27 1.27)) hide)
+    )
+    (property "Datasheet" "~" (id 3) (at 140.97 38.735 0)
+      (effects (font (size 1.27 1.27)) hide)
+    )
+    (property "Mouser Part Number" "604-AA1608ZGSK10MAV " (id 4) (at 140.97 38.735 90)
+      (effects (font (size 1.27 1.27)) hide)
+    )
+    (property "MPN" "Kingbright AA1608ZGSK-10MAV " (id 5) (at 140.97 38.735 90)
+      (effects (font (size 1.27 1.27)) hide)
+    )
+    (pin "1")
+    (pin "2")
+  )
   (symbol (lib_id "AllInOneModule-eagle-import:3.3V") (at 96.52 35.56 0) (unit 1)
     (in_bom yes) (on_board yes)
@@
     (pin "7")
   )
+  (symbol (lib_id "AllInOneModule-eagle-import:GND") (at 140.97 45.085 0) (unit 1)
+    (in_bom yes) (on_board yes)
+    (property "Reference" "#U$0103" (id 0) (at 140.97 45.085 0)
+      (effects (font (size 1.27 1.27)) hide)
+    )
+    (property "Value" "GND" (id 1) (at 139.446 47.625 0)
+      (effects (font (size 1.778 1.5113)) (justify left bottom))
+    )
+    (property "Footprint" "AllInOneModule:" (id 2) (at 140.97 45.085 0)
+      (effects (font (size 1.27 1.27)) hide)
+    )
+    (property "Datasheet" "" (id 3) (at 140.97 45.085 0)
+      (effects (font (size 1.27 1.27)) hide)
+    )
+    (pin "1")
+  )
   (symbol (lib_id "AllInOneModule-eagle-import:CAP_CERAMIC0805-NOOUTLINE") (at 149.86 81.28 0) (unit 1)
     (in_bom yes) (on_board yes)
@@
     (pin "4")
     (pin "5")
+  )
+  (symbol (lib_id "AllInOneModule-eagle-import:3.3V") (at 140.97 22.225 0) (unit 1)
+    (in_bom yes) (on_board yes)
+    (property "Reference" "#U$0102" (id 0) (at 140.97 22.225 0)
+      (effects (font (size 1.27 1.27)) hide)
+    )
+    (property "Value" "3.3V" (id 1) (at 139.446 21.209 0)
+      (effects (font (size 1.27 1.0795)) (justify left bottom))
+    )
+    (property "Footprint" "AllInOneModule:" (id 2) (at 140.97 22.225 0)
+      (effects (font (size 1.27 1.27)) hide)
+    )
+    (property "Datasheet" "" (id 3) (at 140.97 22.225 0)
+      (effects (font (size 1.27 1.27)) hide)
+    )
+    (pin "1")
   )
   (symbol (lib_id "AllInOneModule-eagle-import:GND") (at 149.86 86.36 0) (unit 1)
@@
       (reference "#U$0101") (unit 1) (value "VBAT") (footprint "AllInOneModule:")
     )
+    (path "/d68c5938-5893-4d10-b779-9fd049a30a2b"
+      (reference "#U$0102") (unit 1) (value "3.3V") (footprint "AllInOneModule:")
+    )
+    (path "/9fe61db2-13c8-4b9d-bbde-167454ae1383"
+      (reference "#U$0103") (unit 1) (value "GND") (footprint "AllInOneModule:")
+    )
     (path "/304f094f-1671-4483-b48a-a21534244c3f"
       (reference "C1") (unit 1) (value "10uF") (footprint "Capacitor_SMD:C_0805_2012Metric")
@@
       (reference "D4") (unit 1) (value "S5A") (footprint "Extra:S5AE357T")
     )
+    (path "/816f1b32-6c93-47e7-b628-f143f6ed5263"
+      (reference "D101") (unit 1) (value "POWER") (footprint "LED_SMD:LED_0603_1608Metric")
+    )
     (path "/7b123f12-22af-4a03-98bd-184de6fcc4b8/3840190c-447a-47d0-952a-1be1a49320ea"
       (reference "DI101") (unit 1) (value "KWA-541XVB") (footprint "Displays:KWA-541XVB")
@@
       (reference "R102") (unit 1) (value "10K") (footprint "Resistor_SMD:R_0603_1608Metric")
     )
+    (path "/04fb48c1-c7f4-4fd4-b889-a3fc388cbb74"
+      (reference "R103") (unit 1) (value "30") (footprint "Resistor_SMD:R_0603_1608Metric")
+    )
     (path "/8963df65-c741-4556-b517-67d1c97a55bf"
